File: battery.kicad_sch (KiCad schematic)
At the start: 18 parts, among them Q3 NMOS, Q4 PMOS, Q5 NMOS, Q6 NMOS, SW3 PWR_EN, U6 MCP73831-5-OT, U7 AP9101CK6

Commit message: Updated to 5v power delivery.
Parts:
- removed Q3, Q5, Q6: NMOS, Package_TO_SOT_SMD:SOT-323_SC-70_Handsoldering, symbol Simulation_SPICE:NMOS
- removed Q4: PMOS, Package_TO_SOT_SMD:SOT-323_SC-70_Handsoldering, symbol Simulation_SPICE:PMOS
- added JP14: 5V_PWR, Jumper:SolderJumper-2_P1.3mm_Open_RoundedPad1.0x1.5mm, symbol Jumper:SolderJumper_2_Open
- added Q1, Q2, Q6: BSS84, Package_TO_SOT_SMD:SOT-23_Handsoldering, symbol Transistor_FET:BSS84
- added Q2: MMBT3904, Package_TO_SOT_SMD:SOT-23_Handsoldering, symbol Transistor_BJT:MMBT3904
- added Q7 (x2): BSS138, Package_TO_SOT_SMD:SOT-23_Handsoldering, symbol Transistor_FET:BSS138
- added R38, R39: 330, Resistor_SMD:R_0805_2012Metric_Pad1.20x1.40mm_HandSolder, symbol Device:R_Small
- added R40: 4.7k, Resistor_SMD:R_0805_2012Metric_Pad1.20x1.40mm_HandSolder, symbol Device:R_Small
- D3: footprint LED_SMD:LED_0603_1608Metric_Pad1.05x0.95mm_HandSolder -> LED_SMD:LED_0805_2012Metric_Pad1.15x1.40mm_HandSolder
- SW3: footprint Button_Switch_THT:SW_E-Switch_EG1224_SPDT_Angled -> Button_Switch_THT:SW_CuK_OS102011MA1QN1_SPDT_Angled
Connections:
- net +BATT: now also Q2.3 (D)
- net -BATT: now also Q7.2 (S)
- net GND: now also Q2.2 (E), Q7.2 (S), R39.1
- net VBUS: now also Q2.1 (G)
- net VSYS: now also JP14.1 (A), Q1.3 (D), Q6.2 (S), R40.2
- net VSYS&VBAT: now also Q1.2 (S), Q2.2 (S)
- net at U7.1 (DO): now also Q7.1 (G)
- net at U7.3 (CO): now also Q7.1 (G)
- net PWR_EN renamed 3V3_EN
- net 3V3_EN: now also Q1.1 (G), R38.1
- new net: Q2.1 (B), R38.2, R39.2
- new net: Q7.3 (D), Q7.3 (D)
- new net +5V: JP14.2 (B), Q6.3 (D)
- new net 5V_EN: Q2.3 (C), Q6.1 (G), R40.1
Other:
- moved on the sheet: SW3

Commit message: Updated footprints.
Parts:
- C25: footprint Capacitor_SMD:C_0603_1608Metric_Pad1.08x0.95mm_HandSolder -> Capacitor_SMD:C_0805_2012Metric_Pad1.18x1.45mm_HandSolder
- D2: footprint LED_SMD:LED_0603_1608Metric_Pad1.05x0.95mm_HandSolder -> LED_SMD:LED_0805_2012Metric_Pad1.15x1.40mm_HandSolder
Changed lines of the file:
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@@
       (effects (font (size 1.27 1.27)) (justify left))
     )
-    (property "Footprint" "Capacitor_SMD:C_0603_1608Metric_Pad1.08x0.95mm_HandSolder" (at 157.48 76.2 0)
+    (property "Footprint" "Capacitor_SMD:C_0805_2012Metric_Pad1.18x1.45mm_HandSolder" (at 157.48 76.2 0)
       (effects (font (size 1.27 1.27)) hide)
     )
@@
       (effects (font (size 1.27 1.27)) (justify left))
     )
-    (property "Footprint" "LED_SMD:LED_0603_1608Metric_Pad1.05x0.95mm_HandSolder" (at 50.8 68.58 0)
-      (effects (font (size 1.27 1.27)) hide)
-    )
+    (property "Footprint" "LED_SMD:LED_0805_2012Metric_Pad1.15x1.40mm_HandSolder" (at 50.8 68.58 0)
+      (effects (font (size 1.27 1.27)) hide)
+    )
