File: midi.kicad_sch (KiCad schematic)
At the start: 13 parts, among them J1 MIDIIN, J2 MIDIOUT, J3 MIDIIN, J3 MIDIOUT, Q1 NMOS, U5 6N138

Commit message: Updated to 5v power delivery.
Parts:
- removed Q1: NMOS, Package_TO_SOT_SMD:SOT-323_SC-70_Handsoldering, symbol Simulation_SPICE:NMOS
Connections:
- net +5V: now reaches C19.1, U5.8 (VCC)
Changed lines of the file:
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@@
   (title_block
     (title "pico_synth_sandbox")
-    (date "2023-08-30")
-    (rev "1")
+    (date "2023-09-19")
+    (rev "2")
     (comment 3 "dcdalrymple.com/picosynth/")
     (comment 4 "D Cooper Dalrymple")
@@
   )
   (junction (at 69.85 111.76) (diameter 0) (color 0 0 0 0)
-  )
-  (junction (at 137.16 74.93) (diameter 0) (color 0 0 0 0)
   )
   (junction (at 195.58 111.76) (diameter 0) (color 0 0 0 0)
@@
     (stroke (width 0) (type default))
   )
-  (wire (pts (xy 137.16 74.93) (xy 106.68 74.93))
-    (stroke (width 0) (type default))
-  )
   (wire (pts (xy 204.47 104.14) (xy 203.2 104.14))
     (stroke (width 0) (type default))
@@
     (stroke (width 0) (type default))
   )
+  (wire (pts (xy 137.16 95.25) (xy 137.16 101.6))
+    (stroke (width 0) (type default))
+  )
   (wire (pts (xy 224.79 95.25) (xy 224.79 101.6))
     (stroke (width 0) (type default))
@@
     (stroke (width 0) (type default))
   )
-  (wire (pts (xy 157.48 67.31) (xy 157.48 74.93))
-    (stroke (width 0) (type default))
-  )
   (wire (pts (xy 186.69 104.14) (xy 187.96 104.14))
     (stroke (width 0) (type default))
@@
     (stroke (width 0) (type default))
   )
+  (wire (pts (xy 106.68 95.25) (xy 106.68 99.06))
+    (stroke (width 0) (type default))
+  )
   (wire (pts (xy 186.69 104.14) (xy 186.69 121.92))
     (stroke (width 0) (type default))
   )
-  (wire (pts (xy 142.24 74.93) (xy 137.16 74.93))
-    (stroke (width 0) (type default))
-  )
   (wire (pts (xy 195.58 109.22) (xy 195.58 111.76))
     (stroke (width 0) (type default))
@@
     (stroke (width 0) (type default))
   )
-  (wire (pts (xy 137.16 74.93) (xy 137.16 101.6))
-    (stroke (width 0) (type default))
-  )
   (wire (pts (xy 106.68 111.76) (xy 106.68 113.03))
     (stroke (width 0) (type default))
   )
-  (wire (pts (xy 157.48 74.93) (xy 152.4 74.93))
-    (stroke (width 0) (type default))
-  )
   (wire (pts (xy 52.07 82.55) (xy 52.07 88.9))
     (stroke (width 0) (type default))
@@
   )
   (wire (pts (xy 80.01 101.6) (xy 83.82 101.6))
-    (stroke (width 0) (type default))
-  )
-  (wire (pts (xy 106.68 74.93) (xy 106.68 99.06))
     (stroke (width 0) (type default))
   )
@@
   (text "Midi Output" (at 176.53 66.04 0)
     (effects (font (size 2.54 2.54) (thickness 0.508) bold) (justify left bottom))
-  )
-  (global_label "PWR_EN" (shape input) (at 147.32 67.31 90) (fields_autoplaced)
-    (effects (font (size 1.27 1.27)) (justify left))
-    (property "Intersheetrefs" "${INTERSHEET_REFS}" (at 147.32 56.8863 90)
-      (effects (font (size 1.27 1.27)) (justify left) hide)
-    )
   )
   (global_label "MIDITX" (shape input) (at 185.42 104.14 180) (fields_autoplaced)
@@
     )
   )
-  (symbol (lib_id "pico_synth_sandbox:VSYS") (at 157.48 67.31 0) (mirror y) (unit 1)
-    (in_bom yes) (on_board yes) (dnp no)
-    (property "Reference" "#PWR065" (at 157.48 71.12 0)
-      (effects (font (size 1.27 1.27)) hide)
-    )
-    (property "Value" "VSYS" (at 157.48 62.23 0)
-      (effects (font (size 1.27 1.27)))
-    )
-    (property "Footprint" "" (at 157.48 67.31 0)
-      (effects (font (size 1.27 1.27)) hide)
-    )
-    (property "Datasheet" "" (at 157.48 67.31 0)
-      (effects (font (size 1.27 1.27)) hide)
-    )
-    (pin "1")
-    (instances
-      (project "pico_synth_sandbox"
-        (path "/bfc01388-33ce-4b1a-9d2f-82d750172e5a/d4704e72-f661-4b84-847a-157c0240dc16"
-          (reference "#PWR065") (unit 1)
-        )
-      )
-    )
-  )
   (symbol (lib_id "power:GND") (at 195.58 113.03 0) (unit 1)
     (in_bom yes) (on_board yes) (dnp no) (fields_autoplaced)
-    (property "Reference" "#PWR066" (at 195.58 119.38 0)
+    (property "Reference" "#PWR067" (at 195.58 119.38 0)
       (effects (font (size 1.27 1.27)) hide)
     )
@@
       (project "pico_synth_sandbox"
         (path "/bfc01388-33ce-4b1a-9d2f-82d750172e5a/d4704e72-f661-4b84-847a-157c0240dc16"
-          (reference "#PWR066") (unit 1)
+          (reference "#PWR067") (unit 1)
         )
       )
@@
     )
   )
+  (symbol (lib_id "power:+5V") (at 106.68 95.25 0) (unit 1)
+    (in_bom yes) (on_board yes) (dnp no) (fields_autoplaced)
+    (property "Reference" "#PWR097" (at 106.68 99.06 0)
+      (effects (font (size 1.27 1.27)) hide)
+    )
+    (property "Value" "+5V" (at 106.68 90.17 0)
+      (effects (font (size 1.27 1.27)))
+    )
+    (property "Footprint" "" (at 106.68 95.25 0)
+      (effects (font (size 1.27 1.27)) hide)
+    )
+    (property "Datasheet" "" (at 106.68 95.25 0)
+      (effects (font (size 1.27 1.27)) hide)
+    )
+    (pin "1")
+    (instances
+      (project "pico_synth_sandbox"
+        (path "/bfc01388-33ce-4b1a-9d2f-82d750172e5a/9c12b2ee-f811-4183-acdf-4598ef52f2ef"
+          (reference "#PWR097") (unit 1)
+        )
+        (path "/bfc01388-33ce-4b1a-9d2f-82d750172e5a/d4704e72-f661-4b84-847a-157c0240dc16"
+          (reference "#PWR062") (unit 1)
+        )
+      )
+    )
+  )
   (symbol (lib_id "power:GND") (at 106.68 113.03 0) (unit 1)
     (in_bom yes) (on_board yes) (dnp no) (fields_autoplaced)
-    (property "Reference" "#PWR062" (at 106.68 119.38 0)
+    (property "Reference" "#PWR063" (at 106.68 119.38 0)
       (effects (font (size 1.27 1.27)) hide)
     )
@@
       (project "pico_synth_sandbox"
         (path "/bfc01388-33ce-4b1a-9d2f-82d750172e5a/d4704e72-f661-4b84-847a-157c0240dc16"
-          (reference "#PWR062") (unit 1)
+          (reference "#PWR063") (unit 1)
+        )
+      )
+    )
+  )
+  (symbol (lib_id "power:+5V") (at 137.16 95.25 0) (unit 1)
+    (in_bom yes) (on_board yes) (dnp no) (fields_autoplaced)
+    (property "Reference" "#PWR097" (at 137.16 99.06 0)
+      (effects (font (size 1.27 1.27)) hide)
+    )
+    (property "Value" "+5V" (at 137.16 90.17 0)
+      (effects (font (size 1.27 1.27)))
+    )
+    (property "Footprint" "" (at 137.16 95.25 0)
+      (effects (font (size 1.27 1.27)) hide)
+    )
+    (property "Datasheet" "" (at 137.16 95.25 0)
+      (effects (font (size 1.27 1.27)) hide)
+    )
+    (pin "1")
+    (instances
+      (project "pico_synth_sandbox"
+        (path "/bfc01388-33ce-4b1a-9d2f-82d750172e5a/9c12b2ee-f811-4183-acdf-4598ef52f2ef"
+          (reference "#PWR097") (unit 1)
+        )
+        (path "/bfc01388-33ce-4b1a-9d2f-82d750172e5a/d4704e72-f661-4b84-847a-157c0240dc16"
+          (reference "#PWR065") (unit 1)
         )
       )
@@
         )
         (path "/bfc01388-33ce-4b1a-9d2f-82d750172e5a/d4704e72-f661-4b84-847a-157c0240dc16"
-          (reference "#PWR063") (unit 1)
+          (reference "#PWR064") (unit 1)
         )
       )
@@
   (symbol (lib_id "power:GND") (at 224.79 113.03 0) (unit 1)
     (in_bom yes) (on_board yes) (dnp no) (fields_autoplaced)
-    (property "Reference" "#PWR069" (at 224.79 119.38 0)
+    (property "Reference" "#PWR070" (at 224.79 119.38 0)
       (effects (font (size 1.27 1.27)) hide)
     )
@@
       (project "pico_synth_sandbox"
         (path "/bfc01388-33ce-4b1a-9d2f-82d750172e5a/d4704e72-f661-4b84-847a-157c0240dc16"
-          (reference "#PWR069") (unit 1)
+          (reference "#PWR070") (unit 1)
         )
       )
@@
         )
         (path "/bfc01388-33ce-4b1a-9d2f-82d750172e5a/d4704e72-f661-4b84-847a-157c0240dc16"
-          (reference "#PWR068") (unit 1)
+          (reference "#PWR069") (unit 1)
         )
       )
@@
   (symbol (lib_id "power:GND") (at 137.16 113.03 0) (unit 1)
     (in_bom yes) (on_board yes) (dnp no) (fields_autoplaced)
-    (property "Reference" "#PWR064" (at 137.16 119.38 0)
+    (property "Reference" "#PWR066" (at 137.16 119.38 0)
       (effects (font (size 1.27 1.27)) hide)
     )
@@
       (project "pico_synth_sandbox"
         (path "/bfc01388-33ce-4b1a-9d2f-82d750172e5a/d4704e72-f661-4b84-847a-157c0240dc16"
-          (reference "#PWR064") (unit 1)
+          (reference "#PWR066") (unit 1)
         )
       )
@@
         )
         (path "/bfc01388-33ce-4b1a-9d2f-82d750172e5a/d4704e72-f661-4b84-847a-157c0240dc16"
-          (reference "#PWR067") (unit 1)
+          (reference "#PWR068") (unit 1)
         )
       )
@@
         )
       )
-    )
-  )
-  (symbol (lib_id "Simulation_SPICE:NMOS") (at 147.32 72.39 270) (unit 1)
-    (in_bom yes) (on_board yes) (dnp no) (fields_autoplaced)
-    (property "Reference" "Q1" (at 147.32 78.74 90)
-      (effects (font (size 1.27 1.27)))
-    )
-    (property "Value" "NMOS" (at 147.32 81.28 90)
-      (effects (font (size 1.27 1.27)))
-    )
-    (property "Footprint" "Package_TO_SOT_SMD:SOT-323_SC-70_Handsoldering" (at 149.86 77.47 0)
-      (effects (font (size 1.27 1.27)) hide)
-    )
-    (property "Datasheet" "https://ngspice.sourceforge.io/docs/ngspice-manual.pdf" (at 134.62 72.39 0)
-      (effects (font (size 1.27 1.27)) hide)
-    )
-    (property "Sim.Device" "NMOS" (at 130.175 72.39 0)
-      (effects (font (size 1.27 1.27)) hide)
-    )
-    (property "Sim.Type" "VDMOS" (at 128.27 72.39 0)
-      (effects (font (size 1.27 1.27)) hide)
-    )
-    (property "Sim.Pins" "1=D 2=G 3=S" (at 132.08 72.39 0)
-      (effects (font (size 1.27 1.27)) hide)
-    )
-    (pin "1")
-    (pin "2")
-    (pin "3")
-    (instances
-      (project "pico_synth_sandbox"
-        (path "/bfc01388-33ce-4b1a-9d2f-82d750172e5a/9c12b2ee-f811-4183-acdf-4598ef52f2ef"
-          (reference "Q1") (unit 1)
-        )
-        (path "/bfc01388-33ce-4b1a-9d2f-82d750172e5a/d4704e72-f661-4b84-847a-157c0240dc16"
-          (reference "Q2") (unit 1)
-        )
-      )

Commit message: Updated footprints.
Parts:
- J1: footprint (none) -> LED_SMD:LED_0805_2012Metric_Pad1.15x1.40mm_HandSolder
- R27, R28, R29, R30: footprint Resistor_THT:R_Axial_DIN0204_L3.6mm_D1.6mm_P5.08mm_Horizontal -> Resistor_THT:R_Axial_DIN0207_L6.3mm_D2.5mm_P7.62mm_Horizontal
Changed lines of the file:
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@@
       (effects (font (size 1.27 1.27)))
     )
-    (property "Footprint" "" (at 58.42 99.06 0)
+    (property "Footprint" "LED_SMD:LED_0805_2012Metric_Pad1.15x1.40mm_HandSolder" (at 58.42 99.06 0)
       (effects (font (size 1.27 1.27)) hide)
     )
@@
       (effects (font (size 1.27 1.27)) (justify left))
     )
-    (property "Footprint" "Resistor_THT:R_Axial_DIN0204_L3.6mm_D1.6mm_P5.08mm_Horizontal" (at 106.68 106.68 0)
+    (property "Footprint" "Resistor_THT:R_Axial_DIN0207_L6.3mm_D2.5mm_P7.62mm_Horizontal" (at 106.68 106.68 0)
       (effects (font (size 1.27 1.27)) hide)
     )
@@
       (effects (font (size 1.27 1.27)) (justify left))
     )
-    (property "Footprint" "Resistor_THT:R_Axial_DIN0204_L3.6mm_D1.6mm_P5.08mm_Horizontal" (at 114.3 100.33 0)
+    (property "Footprint" "Resistor_THT:R_Axial_DIN0207_L6.3mm_D2.5mm_P7.62mm_Horizontal" (at 114.3 100.33 0)
       (effects (font (size 1.27 1.27)) hide)
     )
@@
       (effects (font (size 1.27 1.27)) (justify left))
     )
-    (property "Footprint" "Resistor_THT:R_Axial_DIN0204_L3.6mm_D1.6mm_P5.08mm_Horizontal" (at 208.28 100.33 0)
+    (property "Footprint" "Resistor_THT:R_Axial_DIN0207_L6.3mm_D2.5mm_P7.62mm_Horizontal" (at 208.28 100.33 0)
       (effects (font (size 1.27 1.27)) hide)
     )
@@
       (effects (font (size 1.27 1.27)) (justify left))
     )
-    (property "Footprint" "Resistor_THT:R_Axial_DIN0204_L3.6mm_D1.6mm_P5.08mm_Horizontal" (at 46.99 102.87 0)
+    (property "Footprint" "Resistor_THT:R_Axial_DIN0207_L6.3mm_D2.5mm_P7.62mm_Horizontal" (at 46.99 102.87 0)
       (effects (font (size 1.27 1.27)) hide)
     )
